Commit message: Add urdf_to_gmr: generate GMR-ready MuJoCo XML from a robot URDF
- urdf_to_gmr compiles the URDF with MuJoCo's importer, adds a free joint
  on the root link, grounds the robot at qpos=0, keeps fixed links as IK
  frames (+ --frame for extra targets), adds motors/scene/home keyframe and
  writes mesh paths relative to the output (CLI: urdf_to_gmr)
- Rename assets/bdx/mesh -> meshes and fix mesh paths in bdx.urdf/bdx.xml
- Add assets/arti_d1 URDF + meshes with mesh paths fixed (../meshes/)

Co-Authored-By: Claude Opus 5.5 <noreply@anthropic.com>

File: assets/bdx/urdf/bdx.urdf (robot description, URDF)
Before this commit: robot bdx, 21 links, 20 joints
Links:
- link ear_left: geometry collision mesh filename=../meshes/ear_left.stl scale=0.001 0.001 0.001; visual mesh filename=../meshes/ear_left.stl scale=0.001 0.001 0.001
- link ear_right: geometry collision mesh filename=../meshes/ear_right.stl scale=0.001 0.001 0.001; visual mesh filename=../meshes/ear_right.stl scale=0.001 0.001 0.001
- link head_body_pitch: geometry collision mesh filename=../meshes/head_body_pitch.stl scale=0.001 0.001 0.001; visual mesh filename=../meshes/head_body_pitch.stl scale=0.001 0.001 0.001
- link head_body_roll: geometry collision mesh filename=../meshes/head_body_roll.stl scale=0.001 0.001 0.001; visual mesh filename=../meshes/head_body_roll.stl scale=0.001 0.001 0.001
- link head_body_yaw: geometry collision mesh filename=../meshes/head_body_yaw.stl scale=0.001 0.001 0.001; visual mesh filename=../meshes/head_body_yaw.stl scale=0.001 0.001 0.001
- link left_foot_link: geometry collision mesh filename=../meshes/left_foot.stl scale=0.001 0.001 0.001; visual mesh filename=../meshes/left_foot.stl scale=0.001 0.001 0.001
- link left_hip: geometry collision mesh filename=../meshes/left_hip.stl scale=0.001 0.001 0.001; visual mesh filename=../meshes/left_hip.stl scale=0.001 0.001 0.001
- link left_hip_rotation: geometry collision mesh filename=../meshes/left_hip_rotation.stl scale=0.001 0.001 0.001; visual mesh filename=../meshes/left_hip_rotation.stl scale=0.001 0.001 0.001
- link left_shin: geometry collision mesh filename=../meshes/left_shin.stl scale=0.001 0.001 0.001; visual mesh filename=../meshes/left_shin.stl scale=0.001 0.001 0.001
- link left_thigh: geometry collision mesh filename=../meshes/left_thigh.stl scale=0.001 0.001 0.001; visual mesh filename=../meshes/left_thigh.stl scale=0.001 0.001 0.001
- link neck: geometry collision mesh filename=../meshes/neck.stl scale=0.001 0.001 0.001; visual mesh filename=../meshes/neck.stl scale=0.001 0.001 0.001
- link pelvis: geometry collision mesh filename=../meshes/pelvis.stl scale=0.001 0.001 0.001; visual mesh filename=../meshes/pelvis.stl scale=0.001 0.001 0.001
- link right_foot_link: geometry collision mesh filename=../meshes/right_foot.stl scale=0.001 0.001 0.001; visual mesh filename=../meshes/right_foot.stl scale=0.001 0.001 0.001
- link right_hip: geometry collision mesh filename=../meshes/right_hip.stl scale=0.001 0.001 0.001; visual mesh filename=../meshes/right_hip.stl scale=0.001 0.001 0.001
- link right_hip_rotation: geometry collision mesh filename=../meshes/right_hip_rotation.stl scale=0.001 0.001 0.001; visual mesh filename=../meshes/right_hip_rotation.stl scale=0.001 0.001 0.001
- link right_shin: geometry collision mesh filename=../meshes/right_shin.stl scale=0.001 0.001 0.001; visual mesh filename=../meshes/right_shin.stl scale=0.001 0.001 0.001
- link right_thigh: geometry collision mesh filename=../meshes/right_thigh.stl scale=0.001 0.001 0.001; visual mesh filename=../meshes/right_thigh.stl scale=0.001 0.001 0.001
